Commit message: changed head inertia

File: kit_head_description/model/kit_head.gazebo.xacro (robot description, xacro)
@@ -92,4 +92,5 @@
 					<distortionT1>0.0</distortionT1>
 					<distortionT2>0.0</distortionT2>
+					<robotNamespace>${name}</robotNamespace>
 				</plugin>
 			</sensor>
@@ -137,4 +138,5 @@
 					<distortionT1>0.0</distortionT1>
 					<distortionT2>0.0</distortionT2>
+					<robotNamespace>${name}</robotNamespace>
 				</plugin>
 			</sensor>
@@ -149,4 +151,5 @@
 			<sensor type="depth" name="${name}_xtion">
 				<update_rate>10</update_rate>
+<!-- 				<robotNamespace>${name}</robotNamespace>  -->
 				<camera>
 					<horizontal_fov>1.09606677025</horizontal_fov>
@@ -162,4 +165,5 @@
 				</camera>
 				<plugin filename="libgazebo_ros_openni_kinect.so" name="xtion_camera_controller">
+				  <!--libgazebo_ros_openni_kinect.so-->
 					<alwaysOn>true</alwaysOn>
 					<updateRate>10</updateRate>
@@ -172,4 +176,5 @@
 					<frameName>${name}_asus/camera_rgb_optical_frame</frameName>
 					<pointCloudCutoff>0.5</pointCloudCutoff>
+					<pointCloudCutoffMax>3.0</pointCloudCutoffMax>
 					<distortion_k1>0.0</distortion_k1>
 					<distortion_k2>0.0</distortion_k2>
@@ -177,4 +182,9 @@
 					<distortion_t1>0.0</distortion_t1>
 					<distortion_t2>0.0</distortion_t2>
+					<CxPrime>0</CxPrime>
+			                <Cx>0</Cx>
+		 	                <Cy>0</Cy>
+					<focalLength>0.0</focalLength>
+<!-- 					<robotNamespace>${name}</robotNamespace>  -->
 				</plugin>
 			</sensor>

File: kit_head_description/model/kit_head.inertia.xacro (robot description, xacro)
@@ -9,5 +9,5 @@
     <!-- I couldn't make the simulation work with realistic values, so I tweaked the conversion values -->
     <xacro:property name="mm_to_m" value="0.001"/>
-    <xacro:property name="mm2_to_m2" value="0.001"/>
+    <xacro:property name="mm2_to_m2" value="0.01"/>
     <xacro:property name="gr_to_Kg" value="0.001"/>
     <!-- not so negligible, otherwise simulation fails -->
